File: uragon updated/uragon updated.kicad_sch (KiCad schematic)
At the start: 67 parts, among them J1 USB_C_Receptacle_USB2.0_16P, J10 Conn_01x02_Socket, J11 01x07, J2 Conn_01x16_Socket, J3 Conn_01x16_Socket, J4 Conn_01x02_Socket, J5 01x07, J6 01x03, J7 01x03, J8 01x04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

Commit message: Added diodes
Parts:
- removed J11: 01x07, Connector_PinHeader_2.54mm:PinHeader_1x07_P2.54mm_Vertical, symbol Connector:Conn_01x07_Socket
- added D5: SMBJ5.0A, SMBJ5.0A:DIOM4336X265N, symbol SMBJ5.0A:SMBJ5.0A
- added D6: SS54, Diode_SMD:D_SMA, symbol Device:D_Schottky
- added J12: Conn_01x06_Socket, Connector_PinHeader_2.54mm:PinHeader_1x06_P2.54mm_Vertical, symbol Connector:Conn_01x06_Socket
Connections:
- net +5V_LMS: now also J12.1 (Pin_1)
- net +5V_USB: now also D5.A
- net GND: now also D5.C, J12.2 (Pin_2)
- net GPIO12: now also J12.5 (Pin_5)
- net GPIO18: now also J12.6 (Pin_6)
- net GPIO19: now also J12.3 (Pin_3)
- net GPIO21: now also J12.4 (Pin_4)
- net at F2.2, J4.2 (Pin_2): now also D6.1 (K), D6.2 (A)
- no-connect marks 11 -> 10
Other:
- moved on the sheet: F2
